Commit message: simplify orientation

File: nerf_simulation/urdf/camera.xacro (robot description, xacro)
@@ -13,5 +13,5 @@
   <joint name="camera_joint" type="fixed">
     <axis xyz="0 0 0" />
-    <origin xyz="0 0 2" rpy="0 ${PI/6} ${PI/4}"/>
+    <origin xyz="0 0 2" rpy="0 ${PI/6} 0/>
     <parent link="world"/>
     <child link="camera_link"/>

Commit message: missing quote

File: nerf_simulation/urdf/camera.xacro (robot description, xacro)
@@ -13,5 +13,5 @@
   <joint name="camera_joint" type="fixed">
     <axis xyz="0 0 0" />
-    <origin xyz="0 0 2" rpy="0 ${PI/6} 0/>
+    <origin xyz="0 0 2" rpy="0 ${PI/6} 0"/>
     <parent link="world"/>
     <child link="camera_link"/>
